Commit message: Enabled loading of STL files

File: ros2_ws/src/robotic_arm/urdf/arm_assembly.urdf.xacro (robot description, xacro)
@@ -2,5 +2,7 @@
 <robot name="arm_assembly" xmlns:xacro="http://www.ros.org/wiki/xacro">
   <!-- ===== PROPERTIES ===== -->
-  <xacro:property name="package_name" value="robotic_arm" />
+  <xacro:property
+  name="pkg_share"
+  value="$(find robotic_arm)" />
   <!-- Material colors -->
   <material name="blue">
@@ -22,12 +24,12 @@
       <origin xyz="0 0 0" rpy="0 0 0"/>
       <geometry>
-        <mesh filename="package://${package_name}/meshes/base_link.STL"/>
-      </geometry>
-      <material name="blue"/>
-    </visual>
-    <collision>
-      <origin xyz="0 0 0" rpy="0 0 0"/>
-      <geometry>
-        <mesh filename="package://${package_name}/meshes/base_link.STL"/>
+        <mesh filename="file://${pkg_share}/meshes/base_link.STL"/>
+      </geometry>
+      <material name="blue"/>
+    </visual>
+    <collision>
+      <origin xyz="0 0 0" rpy="0 0 0"/>
+      <geometry>
+        <mesh filename="file://${pkg_share}/meshes/base_link.STL"/>
       </geometry>
     </collision>
@@ -45,5 +47,5 @@
       <origin xyz="0 0 0" rpy="0 0 0"/>
       <geometry>
-        <mesh filename="package://${package_name}/meshes/Link_0.STL"/>
+        <mesh filename="file://${pkg_share}/meshes/Link_0.STL"/>
       </geometry>
       <material name="light_blue"/>
@@ -52,5 +54,5 @@
       <origin xyz="0 0 0" rpy="0 0 0"/>
       <geometry>
-        <mesh filename="package://${package_name}/meshes/Link_0.STL"/>
+        <mesh filename="file://${pkg_share}/meshes/Link_0.STL"/>
       </geometry>
     </collision>
@@ -76,12 +78,12 @@
       <origin xyz="0 0 0" rpy="0 0 0"/>
       <geometry>
-        <mesh filename="package://${package_name}/meshes/Link_1.STL"/>
-      </geometry>
-      <material name="blue"/>
-    </visual>
-    <collision>
-      <origin xyz="0 0 0" rpy="0 0 0"/>
-      <geometry>
-        <mesh filename="package://${package_name}/meshes/Link_1.STL"/>
+        <mesh filename="file://${pkg_share}/meshes/Link_1.STL"/>
+      </geometry>
+      <material name="blue"/>
+    </visual>
+    <collision>
+      <origin xyz="0 0 0" rpy="0 0 0"/>
+      <geometry>
+        <mesh filename="file://${pkg_share}/meshes/Link_1.STL"/>
       </geometry>
     </collision>
@@ -107,12 +109,12 @@
       <origin xyz="0 0 0" rpy="0 0 0"/>
       <geometry>
-        <mesh filename="package://${package_name}/meshes/Link_2.STL"/>
-      </geometry>
-      <material name="blue"/>
-    </visual>
-    <collision>
-      <origin xyz="0 0 0" rpy="0 0 0"/>
-      <geometry>
-        <mesh filename="package://${package_name}/meshes/Link_2.STL"/>
+        <mesh filename="file://${pkg_share}/meshes/Link_2.STL"/>
+      </geometry>
+      <material name="blue"/>
+    </visual>
+    <collision>
+      <origin xyz="0 0 0" rpy="0 0 0"/>
+      <geometry>
+        <mesh filename="file://${pkg_share}/meshes/Link_2.STL"/>
       </geometry>
     </collision>
@@ -138,12 +140,12 @@
       <origin xyz="0 0 0" rpy="0 0 0"/>
       <geometry>
-        <mesh filename="package://${package_name}/meshes/Link_3.STL"/>
-      </geometry>
-      <material name="blue"/>
-    </visual>
-    <collision>
-      <origin xyz="0 0 0" rpy="0 0 0"/>
-      <geometry>
-        <mesh filename="package://${package_name}/meshes/Link_3.STL"/>
+        <mesh filename="file://${pkg_share}/meshes/Link_3.STL"/>
+      </geometry>
+      <material name="blue"/>
+    </visual>
+    <collision>
+      <origin xyz="0 0 0" rpy="0 0 0"/>
+      <geometry>
+        <mesh filename="file://${pkg_share}/meshes/Link_3.STL"/>
       </geometry>
     </collision>
@@ -169,12 +171,12 @@
       <origin xyz="0 0 0" rpy="0 0 0"/>
       <geometry>
-        <mesh filename="package://${package_name}/meshes/Link_4.STL"/>
-      </geometry>
-      <material name="blue"/>
-    </visual>
-    <collision>
-      <origin xyz="0 0 0" rpy="0 0 0"/>
-      <geometry>
-        <mesh filename="package://${package_name}/meshes/Link_4.STL"/>
+        <mesh filename="file://${pkg_share}/meshes/Link_4.STL"/>
+      </geometry>
+      <material name="blue"/>
+    </visual>
+    <collision>
+      <origin xyz="0 0 0" rpy="0 0 0"/>
+      <geometry>
+        <mesh filename="file://${pkg_share}/meshes/Link_4.STL"/>
       </geometry>
     </collision>
