Commit message: Cloned cobot tutorial

File: ros2_ws/src/mycobot_ros2/mycobot_description/urdf/robots/mycobot_280.urdf.xacro (robot description, xacro)
@@ -44,6 +44,5 @@
         </xacro:if>
     </xacro:if>
-    <!--commented out the below so that program could run > -->
-    <!-- <xacro:include filename="$(find mycobot_description)/urdf/control/gazebo_sim_ros2_control.urdf.xacro" />
+    <xacro:include filename="$(find mycobot_description)/urdf/control/gazebo_sim_ros2_control.urdf.xacro" />
     <xacro:load_gazebo_sim_ros2_control_plugin
       robot_name="$(arg robot_name)"
@@ -53,5 +52,5 @@
       prefix="$(arg prefix)"
       flange_link="$(arg flange_link)"
-      use_gazebo="$(arg use_gazebo)"/> -->
-    <xacro:include filename="$(find mycobot_description)/meshes/urdf/sensors/intel_rgbd_cam_d435.urdf.xacro"/>
+      use_gazebo="$(arg use_gazebo)"/>
+    <xacro:include filename="$(find mycobot_description)/urdf/sensors/intel_rgbd_cam_d435.urdf.xacro"/>
 </robot>

File: ros2_ws/src/robotic_arm/urdf/arm_assembly.urdf.xacro (robot description, xacro)
@@ -16,5 +16,5 @@
     <inertial>
       <origin xyz="-0.00079815 0.0029373 -1.9921E-05" rpy="0 0 0"/>
-      <mass value="0.3171"/>
+      <mass value="2"/>
       <inertia
         ixx="0.0002369" ixy="2.2819E-07" ixz="-1.3738E-07"
@@ -39,5 +39,5 @@
     <inertial>
       <origin xyz="0.0396837 0.028045 -3.8214E-07" rpy="0 0 0"/>
-      <mass value="0.332338"/>
+      <mass value="2"/>
       <inertia
         ixx="0.00056310" ixy="-0.00012714" ixz="-1.3669E-09"
@@ -70,5 +70,5 @@
     <inertial>
       <origin xyz="-0.163682 1.0326E-06 -0.0053131" rpy="0 0 0"/>
-      <mass value="1.29152"/>
+      <mass value="2"/>
       <inertia
         ixx="0.0015238" ixy="2.4811E-08" ixz="6.2596E-06"
@@ -101,5 +101,5 @@
     <inertial>
       <origin xyz="-0.041346 0.084874 -0.016207" rpy="0 0 0"/>
-      <mass value="0.400209"/>
+      <mass value="2"/>
       <inertia
         ixx="0.00051636" ixy="8.1074E-05" ixz="4.0861E-06"
@@ -132,5 +132,5 @@
     <inertial>
       <origin xyz="-0.266602 0.028901 -0.00045148" rpy="0 0 0"/>
-      <mass value="0.455178"/>
+      <mass value="2"/>
       <inertia
         ixx="0.00025930" ixy="3.8430E-05" ixz="5.0616E-07"
@@ -163,5 +163,5 @@
     <inertial>
       <origin xyz="-0.028470 -0.036145 -0.021734" rpy="0 0 0"/>
-      <mass value="0.097487"/>
+      <mass value="2"/>
       <inertia
         ixx="3.4201E-05" ixy="-7.8453E-06" ixz="-1.5867E-06"
