Commit message: Made rviz config file

File: ros2_ws/src/arm_description/urdf/arm.xacro (robot description, xacro)
@@ -35,5 +35,5 @@
   <link name="Link_0">
     <inertial>
-      <origin xyz="0.0396837 0.028045 -3.8214E-07" rpy="0 0 0"/>
+      <origin xyz="0.0396837 0.028045 1" rpy="0 0 0"/>
       <mass value="2"/>
       <inertia
