Commit message: Debugged controller manager launch code

File: ros2_ws/src/arm_description/urdf/kipp.ros2_control.xacro (robot description, xacro)
@@ -1,6 +1,4 @@
 <?xml version="1.0"?>
 <robot xmlns:xacro="http://www.ros.org/wiki/xacro">
-    <xacro:macro name="kipp_ros2_control" params="name initial_positions_file">
-        <xacro:property name="initial_positions" value="${load_yaml(initial_positions_file)['initial_positions']}"/>
         <ros2_control name="Arm" type="system">
             <hardware>
@@ -39,4 +37,3 @@
             </joint>
         </ros2_control>
-    </xacro:macro>
 </robot>
